File: controller_mb_usb.kicad_pcb (KiCad board)
At the start: 2 copper layers, 115 x 68 mm, 48 parts, among them J1 AVR-ISP-6, J2 Conn_01x19, J3 CAN, J4 USB_B, U1 AP5100, U2 MCP2551-I-SN, U3 ATmega16M1-AU, U4 ADuM121N, U5 FT230XS, U6 ADuM121N, Y1 12MHz

Commit message: Init v0.2
Parts:
- removed the C5 at (120.7, 100.3)
- removed the C6 at (120.7, 103.5)
- removed the D2 at (120.7, 94.6)
- removed the L1 at (115.6, 80.0)
- removed L2: 33uH, Inductor_SMD:L_10.4x10.4_H4.8
- removed the R1 at (120.7, 82.5)
- removed the R2 at (127.0, 90.2)
- removed the R3 at (127.0, 83.8)
- added JP2: Jumper_NC_Small, Jumper:SolderJumper-2_P1.3mm_Open_Pad1.0x1.5mm, F.Cu at (172.9, 86.3)
- added JP3: Shield, Jumper:SolderJumper-2_P1.3mm_Open_Pad1.0x1.5mm, F.Cu at (187.7, 64.0)
- C1: value 22nF -> 100uF; footprint Capacitor_SMD:C_1206_3216Metric_Pad1.42x1.75mm_HandSolder -> Capacitor_THT:CP_Radial_D6.3mm_P2.50mm
- C3: value 10uF -> 100nF
- C4: value 100pF -> 47uF; footprint Capacitor_SMD:C_1206_3216Metric_Pad1.42x1.75mm_HandSolder -> Capacitor_THT:CP_Radial_D6.3mm_P2.50mm
- J2: value Conn_01x19 -> Front panel
- JP1: footprint Connector_PinHeader_2.54mm:PinHeader_1x02_P2.54mm_Vertical -> Jumper:SolderJumper-2_P1.3mm_Open_Pad1.0x1.5mm
- U1: value AP5100 -> LM78M05; footprint Package_TO_SOT_SMD:SOT-23-6 -> Package_TO_SOT_SMD:TO-252-2
- U3: value ATmega16M1-AU -> ATmega32M1-AU
- moved C3 15.0 mm to (116.8, 99.6)
- moved C4 14.6 mm to (127.9, 104.7)
- moved C1 12.2 mm to (115.2, 80.5), turned to 0 degrees
- moved C2 10.5 mm to (116.5, 86.9)
- moved U1 5.24 mm to (119.0, 93.2), turned to 0 degrees
- moved JP1 3.57 mm to (134.3, 69.5), turned to 180 degrees
- moved J4 2.10 mm to (197.7, 68.0)
- moved J3 2.00 mm to (120.0, 64.0)
- moved G*** 1.35 mm to (116.9, 116.4)
- renumbered C12 to C10, C13 to C11, C14 to C12, C15 to C13, C16 to C14, C17 to C15, C18 to C16, C19 to C17, C20 to C18, C21 to C19, C22 to C20, C7 to C5, C8 to C6, C9 to C7, C10 to C8, C11 to C9, D3 to D2, L3 to L1, R4 to R1, R5 to R2, R6 to R3, R7 to R4
Connections:
- C1 pad 2: Net-(C1-Pad2) -> GND
- C2 pad 1: Net-(C2-Pad1) -> Net-(C1-Pad1)
- C3 pad 1: Net-(C3-Pad1) -> +5V
- C4 pad 2: /FB -> GND
- D1 pad 1: Net-(C2-Pad1) -> Net-(C1-Pad1)
- J4 pad 5: GNDD -> Net-(J4-Pad5)
- U1 pad 3: /FB -> +5V
- U4 pad 2: /SCK(RX) -> Net-(JP2-Pad1)
Routing:
- net Net-(J3-Pad0): track 9.68 -> 39.9 mm
- net GND: track 50.8 -> 30.6 mm, vias 12 -> 33
- net Net-(C1-Pad1): track 2.39 -> 20.6 mm
- net Net-(J4-Pad5): track 0.00 -> 17.3 mm
- net +5V: track 264.9 -> 248.2 mm
- net Net-(C2-Pad1): track 13.0 -> 0.00 mm
- net /FB: track 11.0 -> 0.00 mm, vias 2 -> 0
- net /SCK(RX): track 43.3 -> 35.5 mm
- net Net-(JP2-Pad1): track 0.00 -> 6.53 mm
- net Net-(R1-Pad2): track 5.96 -> 0.00 mm
- net GNDD: track 24.7 -> 28.2 mm
- net /D+: track 12.1 -> 14.7 mm
- net /CAN_H: track 30.9 -> 31.8 mm
- net Net-(C20-Pad1): track 14.9 -> 15.8 mm
- net /CAN_L: track 34.5 -> 35.4 mm
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- removed copper zone on F.Cu, net +5V
- removed copper zone on F.Cu, net Net-(C1-Pad2)
- removed copper zone on F.Cu, net Net-(C3-Pad1)
Other:
- board size 115 x 68 mm -> 115 x 69.8 mm
- board text added: "H9 controller main board with USB v0.2 by SQ8KFH"
- board text added: "Low Ground Shield High Power (max 15V)"
- board text removed: "H9 controller main board with USB v0.1 by SQ8KFH"
- board text removed: "Low Ground Shield High Power (max 20V)"

Commit message: v0.2
Other:
- board text added: "H9 controller main board with a USB v0.2 by SQ8KFH"
- board text removed: "H9 controller main board with USB v0.2 by SQ8KFH"
Changed lines of the file:
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@@
   (page A4)
   (title_block
-    (title "H9 controller main board with USB")
+    (title "H9 controller main board with a USB")
     (date 2020-12-21)
     (rev 0.2)
@@
   )
   (setup
-    (last_trace_width 0.508)
+    (last_trace_width 0.3048)
     (user_trace_width 0.508)
     (trace_clearance 0.2286)
@@
     (add_net "Net-(D1-Pad2)")
     (add_net "Net-(J3-Pad0)")
-    (add_net "Net-(J3-Pad1)")
-    (add_net "Net-(J3-Pad4)")
     (add_net "Net-(J3-Pad5)")
-    (add_net "Net-(J3-Pad6)")
-    (add_net "Net-(J3-Pad8)")
     (add_net "Net-(J4-Pad5)")
     (add_net "Net-(JP2-Pad1)")
     (add_net "Net-(R1-Pad1)")
-    (add_net "Net-(U2-Pad5)")
-    (add_net "Net-(U3-Pad21)")
     (add_net "Net-(U4-Pad6)")
     (add_net "Net-(U4-Pad7)")
-    (add_net "Net-(U5-Pad14)")
-    (add_net "Net-(U5-Pad15)")
-    (add_net "Net-(U5-Pad16)")
     (add_net "Net-(U5-Pad2)")
     (add_net "Net-(U5-Pad6)")
-    (add_net "Net-(U5-Pad7)")
   )
   (module Jumper:SolderJumper-2_P1.3mm_Open_Pad1.0x1.5mm (layer F.Cu)
@@
   (gr_line (start 102.5 58) (end 102.5 55.2) (layer Edge.Cuts) (width 0.05))
   (gr_line (start 100 58) (end 102.5 58) (layer Edge.Cuts) (width 0.05))
-  (gr_text "H9 controller main board\nwith USB v0.2\nby SQ8KFH" (at 197.79 116.364) (layer F.SilkS)
+  (gr_text "H9 controller main board\nwith a USB v0.2\nby SQ8KFH" (at 197.79 116.364) (layer F.SilkS)
     (effects (font (size 1.5 1.5) (thickness 0.2)))
   )
